Commit message: updated model configuration

File: hydrofoil_usv_description/urdf/hydrofoil.urdf (robot description, URDF)
Before this commit: robot hydrofoil, 1 links, 0 joints
Links:
- link base_link: geometry collision box size=12.5 4.7 2.2; visual mesh filename=package://hydrofoil_usv_description/models/hydrofoil_vessel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
