Commit message: renamed project and updated visualizer

File: urdf/hydrofoil.urdf (robot description, URDF)
Before this commit: robot hydrofoil, 1 links, 0 joints
Links:
- link base_link: geometry collision box size=12.5 4.7 2.2; visual mesh filename=package://hybraut_nav_colreg_sim/models/hydrofoil_vessel/me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
